File: DAQ-KICAD/DAQ-Bicineta/DAQ-Bicineta.kicad_pcb (KiCad board)
At the start: 2 copper layers, 100 x 100 mm, 17 parts, among them U3 ESP32-DEVKIT-V1

Commit message: DAQ-V2-KICAD-modification
Parts:
- removed the G*** at (149.5, 63.0)
- added 10kOhm: R, Connector_PinSocket_2.54mm:PinSocket_1x02_P2.54mm_Vertical, F.Cu at (174.5, 94.8)
- added 1kOhm: R, Connector_PinSocket_2.54mm:PinSocket_1x02_P2.54mm_Vertical, F.Cu at (122.4, 128.8)
- added 1kOhm: R, Connector_PinSocket_2.54mm:PinSocket_1x02_P2.54mm_Vertical, F.Cu at (174.5, 106.3)
- added 1kOhm: R, Connector_PinSocket_2.54mm:PinSocket_1x02_P2.54mm_Vertical, F.Cu at (122.4, 118.3)
- added ACS712_2: Conn_01x03, Connector_PinSocket_2.54mm:PinSocket_1x03_P2.54mm_Vertical, F.Cu at (115.1, 81.9)
- added ACS712_3: Conn_01x03, Connector_PinSocket_2.54mm:PinSocket_1x03_P2.54mm_Vertical, F.Cu at (126.2, 81.9)
- added ACS712_4: Conn_01x03, Connector_PinSocket_2.54mm:PinSocket_1x03_P2.54mm_Vertical, F.Cu at (119.6, 96.1)
- added Accelerator: Conn_01x02, Connector_PinSocket_2.54mm:PinSocket_1x02_P2.54mm_Vertical, F.Cu at (107.6, 129.9)
- added C-68nF1: C_Small, Connector_PinSocket_2.54mm:PinSocket_1x02_P2.54mm_Vertical, F.Cu at (122.3, 104.9)
- added G***: LOGO, Images:GCA_Shield_Logo2, F.Cu at (150.1, 62.2)
- added G***: LOGO, Images:GCA_Shield_Logo, B.Cu at (150.4, 100.1)
- added LM324: Conn_02x07_Odd_Even, MyPrintFoot:LM324, F.Cu at (180.3, 135.6)
- KY-24: footprint Connector_PinSocket_2.54mm:PinSocket_1x04_P2.54mm_Horizontal -> Connector_PinSocket_2.54mm:PinSocket_1x04_P2.54mm_Vertical
- MicroSD: renamed from MicroSD1; footprint Connector_PinSocket_2.54mm:PinSocket_1x06_P2.54mm_Horizontal -> Connector_PinSocket_2.54mm:PinSocket_1x06_P2.54mm_Vertical
- moved MicroSD 20.8 mm to (193.3, 107.8)
- moved GPS 20.2 mm to (107.1, 121.0)
- moved T-D500 18.6 mm to (190.7, 115.4)
- moved ACS712_1 15.9 mm to (103.9, 81.9)
- moved KY-24 13.4 mm to (107.2, 100.0)
- moved 300kOhm 6.84 mm to (174.5, 120.1), turned to 180 degrees
- moved PowerModule1 4.73 mm to (190.4, 83.0)
- renumbered R-150k to 300kOhm, ACS712 to ACS712_1, GPS1 to GPS
Connections:
- net CS_OUT renamed CS_OUT_1
- 300kOhm pad 1: CS_VCC -> Net-(LM324-Pin_3)
- 300kOhm pad 2: T-D500_OUT -> ACCELERATOR_GND
- ACS712_1 pad 3: CS_GND -> ACCELERATOR_GND
- GPS pad 1: CS_GND -> ACCELERATOR_GND
- GPS pad 4: GPS_VCC -> CS_VCC
- H1 pad 1: CS_GND -> ACCELERATOR_GND
- H2 pad 2: CS_GND -> ACCELERATOR_GND
- H3 pad 3: CS_GND -> ACCELERATOR_GND
- H4 pad 4: CS_GND -> ACCELERATOR_GND
- KY-24 pad 2: CS_GND -> ACCELERATOR_GND
- KY-24 pad 3: GPS_VCC -> CS_VCC
- MicroSD pad 5: GPS_VCC -> CS_VCC
- MicroSD pad 6: CS_GND -> ACCELERATOR_GND
- PowerModule1 pad 1: GPS_VCC -> CS_VCC
- PowerModule1 pad 2: GPS_VCC -> CS_VCC
- PowerModule1 pad 5: CS_GND -> ACCELERATOR_GND
- PowerModule1 pad 6: CS_GND -> ACCELERATOR_GND
- T-D500 pad 1: T-D500_OUT -> Net-(LM324-Pin_3)
- T-D500 pad 2: CS_GND -> T-D500_OUT
- U3 pad 1: CS_VCC -> T-D500_VCC
- U3 pad 2: CS_GND -> ACCELERATOR_GND
- U3 pad 23: unconnected-(U3-D25-Pad23) -> ACCELERATOR_Vout
- U3 pad 26: unconnected-(U3-D14-Pad26) -> CS_OUT_4
- U3 pad 27: unconnected-(U3-D12-Pad27) -> CS_OUT_2
- U3 pad 28: unconnected-(U3-D13-Pad28) -> CS_OUT_3
- U3 pad 29: CS_GND -> ACCELERATOR_GND
- U3 pad 30: GPS_VCC -> CS_VCC
Routing:
- net GPS_VCC: track 223.3 -> 0.00 mm, vias 4 -> 0
- net T-D500_VCC: track 0.00 -> 163.3 mm, vias 0 -> 2
- net CS_VCC: track 109.8 -> 211.7 mm
- net ACCELERATOR_Vout: track 0.00 -> 69.4 mm
- net MSD_MISO: track 89.9 -> 153.0 mm
- net CS_OUT_2: track 0.00 -> 54.6 mm, vias 0 -> 2
- net CS_OUT_4: track 0.00 -> 49.5 mm, vias 0 -> 1
- net CS_OUT_3: track 0.00 -> 43.1 mm
- net Net-(LM324-Pin_5): track 0.00 -> 41.1 mm, vias 0 -> 1
- net Net-(LM324-Pin_3): track 0.00 -> 37.4 mm, vias 0 -> 3
- net KY_DO: track 104.3 -> 71.4 mm, vias 2 -> 0
- net MSD_MOSI: track 66.4 -> 94.0 mm, vias 2 -> 1
- net MSD_SCK: track 93.1 -> 118.1 mm
- net MSD_CS: track 96.3 -> 72.4 mm
- net PM_I: track 66.7 -> 45.0 mm, vias 1 -> 0
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- added copper zone on B.Cu, net ACCELERATOR_GND
- added copper zone on F.Cu, net ACCELERATOR_GND
- removed copper zone on B.Cu, net CS_GND
- removed copper zone on F.Cu, net CS_GND
